Commit message: fixing URDF

File: anubis_ws/src/moveit_servo/config/urdf/braccio.urdf (robot description, URDF)
Before this commit: robot visual, 9 links, 8 joints
Links:
- link gripper_base: geometry visual mesh filename=package://moveit_servo/config/meshes/gripper_base.stl
- link gripper_fix: geometry visual mesh filename=package://moveit_servo/config/meshes/gripper_fix.stl
- link gripper_movable: geometry visual mesh filename=package://moveit_servo/config/meshes/gripper_movable.stl
- link link1: geometry visual mesh filename=package://moveit_servo/config/meshes/base.stl
- link link2: geometry visual mesh filename=package://moveit_servo/config/meshes/shoulder.stl
- link link3: geometry visual mesh filename=package://moveit_servo/config/meshes/elbow.stl
- link link4: geometry visual mesh filename=package://moveit_servo/config/meshes/wrist_pitch.stl
- link link5: geometry visual mesh filename=package://moveit_servo/config/meshes/wrist_roll.stl
