Commit message: working but not controllable

File: anubis_ws/src/moveit_servo/config/urdf/braccio_arm.urdf (robot description, URDF)
Before this commit: robot visual, 8 links, 7 joints
Links:
- added link fake_wrist_link, mass 0.001
Joints:
- added joint fake_wrist_joint: type revolute, parent wrist_roll_link, child fake_wrist_link, origin xyz=0 0 0 rpy=0 0 0, axis 0 0 1, limit lower=-3.1416 upper=3.1416 effort=0.1 velocity=5.0
